Commit message: test gazebo

File: urdf/bioroid.urdf (robot description, URDF)
Before this commit: robot bioloid, 55 links, 54 joints
Links:
- link base_link: mass None -> 1

Commit message: test gazebo

File: urdf/bioroid.urdf (robot description, URDF)
Before this commit: robot bioloid, 55 links, 54 joints
Links:
- link arm_joint_left: mass None -> 1
- link arm_joint_right: mass None -> 1
- link d1: mass None -> 1
- link d10: mass None -> 1
- link d10_join: mass None -> 1
- link d11: mass None -> 1
- link d11_join: mass None -> 1
- link d12: mass None -> 1
- link d12_join: mass None -> 1
- link d13: mass None -> 1
- link d13_join: mass None -> 1
- link d14: mass None -> 1
- link d14_join: mass None -> 1
- link d15: mass None -> 1
- link d15_join: mass None -> 1
- link d16: mass None -> 1
- link d16_join: mass None -> 1
- link d17: mass None -> 1
- link d17_join: mass None -> 1
- link d18: mass None -> 1
- link d18_join: mass None -> 1
- link d1_join: mass None -> 1
- link d2: mass None -> 1
- link d2_join: mass None -> 1
- link d3: mass None -> 1
- link d3_join: mass None -> 1
- link d4: mass None -> 1
- link d4_join: mass None -> 1
- link d5_join: mass None -> 1
- link d6: mass None -> 1
- link d6_join: mass None -> 1
- link d7: mass None -> 1
- link d7_join: mass None -> 1
- link d8: mass None -> 1
- link d8_join: mass None -> 1
- link d9: mass None -> 1
- link d9_join: mass None -> 1
- link feet_join_left: mass None -> 1
- link feet_join_right: mass None -> 1
- link feet_left: mass None -> 1
- link feet_right: mass None -> 1
- link head: mass None -> 1
- link low_femur_left: mass None -> 1
- link low_femur_right: mass None -> 1
- link mid_femur_left: mass None -> 1
- link mid_femur_right: mass None -> 1
- link pelvis: mass None -> 1
- link shoulder_left: mass None -> 1
- link shoulder_right: mass None -> 1
- link tibia_left: mass None -> 1
- link tibia_right: mass None -> 1
- link upper_femur_left: mass None -> 1
- link upper_femur_right: mass None -> 1
